Commit message: Merged changes from December backup

File: kinova_description/urdf/j2s6s200.xacro (robot description, xacro)
@@ -1,4 +1,4 @@
 <?xml version="1.0"?>
-<!-- j2_n7 refers to jaco v2 7DOF non-spherical -->
+<!-- j2_6s refers to jaco v2 6DOF spherical -->
 <root xmlns:xi="http://www.w3.org/2001/XInclude"
     xmlns:gazebo="http://playerstage.sourceforge.net/gazebo/xmlschema/#gz"
@@ -20,10 +20,9 @@
     <xacro:property name="link_base_mesh" value="base" />
     <xacro:property name="link_1_mesh" value="shoulder" />
-    <xacro:property name="link_2_mesh" value="arm_half_1" />
-    <xacro:property name="link_3_mesh" value="arm_half_2" />
-    <xacro:property name="link_4_mesh" value="forearm" />
-    <xacro:property name="link_5_mesh" value="wrist" />
-    <xacro:property name="link_6_mesh" value="wrist" />
-    <xacro:property name="link_7_mesh" value="hand_3finger" />
+    <xacro:property name="link_2_mesh" value="arm" />
+    <xacro:property name="link_3_mesh" value="forearm" />
+    <xacro:property name="link_4_mesh" value="wrist_spherical_1" />
+    <xacro:property name="link_5_mesh" value="wrist_spherical_2" />
+    <xacro:property name="link_6_mesh" value="hand_2finger" />
     <!--Used for conditional arguments for setting inertial parameters
         base 0, shoulder 1, arm 2, forearm 3, wrist 4, arm_mico 5,
@@ -34,10 +33,9 @@
     <xacro:property name="link_base_mesh_no" value="0" />
     <xacro:property name="link_1_mesh_no" value="1" />
-    <xacro:property name="link_2_mesh_no" value="6" />
-    <xacro:property name="link_3_mesh_no" value="7" />
-    <xacro:property name="link_4_mesh_no" value="3" />
-    <xacro:property name="link_5_mesh_no" value="4" />
-    <xacro:property name="link_6_mesh_no" value="4" />
-    <xacro:property name="link_7_mesh_no" value="55" />
+    <xacro:property name="link_2_mesh_no" value="2" />
+    <xacro:property name="link_3_mesh_no" value="3" />
+    <xacro:property name="link_4_mesh_no" value="8" />
+    <xacro:property name="link_5_mesh_no" value="9" />
+    <xacro:property name="link_6_mesh_no" value="55" />
     <xacro:property name="joint_base" value="joint_base" />
     <xacro:property name="joint_base_type" value="fixed" />
@@ -58,34 +56,34 @@
     <xacro:property name="joint_2_axis_xyz" value="0 0 1" />
     <xacro:property name="joint_2_origin_xyz" value="0 0.0016 -0.11875" />
-    <xacro:property name="joint_2_origin_rpy" value="-${J_PI/2} 0 ${J_PI}" />
-    <xacro:property name="joint_2_lower_limit" value="${30/180*J_PI}" />
-    <xacro:property name="joint_2_upper_limit" value="${330/180*J_PI}" />
+    <xacro:property name="joint_2_origin_rpy" value="${-J_PI/2} 0 ${J_PI}"/>
+    <xacro:property name="joint_2_lower_limit" value="${47/180*J_PI}" />
+    <xacro:property name="joint_2_upper_limit" value="${313/180*J_PI}" />
     <xacro:property name="joint_2_velocity_limit" value="${36*J_PI/180}" />
     <xacro:property name="joint_2_torque_limit" value="80" />
     <xacro:property name="joint_3" value="joint_3" />
-    <xacro:property name="joint_3_type" value="continuous" />
+    <xacro:property name="joint_3_type" value="revolute" />
     <xacro:property name="joint_3_axis_xyz" value="0 0 1" />
-    <xacro:property name="joint_3_origin_xyz" value="0 -0.205 0" />
-    <xacro:property name="joint_3_origin_rpy" value="${J_PI/2} 0 ${J_PI}" />
-    <xacro:property name="joint_3_lower_limit" value="${-5*J_PI/4}" />
-    <xacro:property name="joint_3_upper_limit" value="${1*J_PI/4}" />
+    <xacro:property name="joint_3_origin_xyz" value="0 -0.410 0" />
+    <xacro:property name="joint_3_origin_rpy" value="0 ${J_PI} 0" />
+    <xacro:property name="joint_3_lower_limit" value="${19/180*J_PI}" />
+    <xacro:property name="joint_3_upper_limit" value="${341/180*J_PI}" />
     <xacro:property name="joint_3_velocity_limit" value="${36*J_PI/180}" />
     <xacro:property name="joint_3_torque_limit" value="40" />
     <xacro:property name="joint_4" value="joint_4" />
-    <xacro:property name="joint_4_type" value="revolute" />
+    <xacro:property name="joint_4_type" value="continuous" />
     <xacro:property name="joint_4_axis_xyz" value="0 0 1" />
-    <xacro:property name="joint_4_origin_xyz" value="0 0 -0.205" />
-    <xacro:property name="joint_4_origin_rpy" value="${J_PI/2} 0 ${J_PI}" />
-    <xacro:property name="joint_4_lower_limit" value="${30/180*J_PI}" />
-    <xacro:property name="joint_4_upper_limit" value="${330/180*J_PI}" />
-    <xacro:property name="joint_4_velocity_limit" value="${36*J_PI/180}" />
-    <xacro:property name="joint_4_torque_limit" value="40" />
+    <xacro:property name="joint_4_origin_xyz" value="0 0.2073 -0.0114" />
+    <xacro:property name="joint_4_origin_rpy" value="${-J_PI/2} 0 ${J_PI}" />
+    <xacro:property name="joint_4_lower_limit" value="${-2*J_PI}" />
+    <xacro:property name="joint_4_upper_limit" value="${2*J_PI}" />
+    <xacro:property name="joint_4_velocity_limit" value="${48*J_PI/180}" />
+    <xacro:property name="joint_4_torque_limit" value="20" />
     <xacro:property name="joint_5" value="joint_5" />
-    <xacro:property name="joint_5_type" value="continuous" />
+    <xacro:property name="joint_5_type" value="revolute" />
     <xacro:property name="joint_5_axis_xyz" value="0 0 1" />
-    <xacro:property name="joint_5_origin_xyz" value="0 0.2073 -0.0114" />
-    <xacro:property name="joint_5_origin_rpy" value="${-J_PI/2} 0 ${J_PI}" />
-    <xacro:property name="joint_5_lower_limit" value="${-2*J_PI}" />
-    <xacro:property name="joint_5_upper_limit" value="${2*J_PI}" />
+    <xacro:property name="joint_5_origin_xyz" value="0 0 -0.10375" />
+    <xacro:property name="joint_5_origin_rpy" value="${J_PI/2} 0 ${J_PI}" />
+    <xacro:property name="joint_5_lower_limit" value="${30/180*J_PI}" />
+    <xacro:property name="joint_5_upper_limit" value="${330/180*J_PI}" />
     <xacro:property name="joint_5_velocity_limit" value="${48*J_PI/180}" />
     <xacro:property name="joint_5_torque_limit" value="20" />
@@ -93,19 +91,10 @@
     <xacro:property name="joint_6_type" value="continuous" />
     <xacro:property name="joint_6_axis_xyz" value="0 0 1" />
-    <xacro:property name="joint_6_origin_xyz" value="0 -0.03703 -0.06414" />
-    <xacro:property name="joint_6_origin_rpy" value="${J_PI/3} 0 ${J_PI}" />
+    <xacro:property name="joint_6_origin_xyz" value="0 0.10375 0" />
+    <xacro:property name="joint_6_origin_rpy" value="${-J_PI/2} 0 ${J_PI}" />
     <xacro:property name="joint_6_lower_limit" value="${-2*J_PI}" />
     <xacro:property name="joint_6_upper_limit" value="${2*J_PI}" />
     <xacro:property name="joint_6_velocity_limit" value="${48*J_PI/180}" />
     <xacro:property name="joint_6_torque_limit" value="20" />
-    <xacro:property name="joint_7" value="joint_7" />
-    <xacro:property name="joint_7_type" value="continuous" />
-    <xacro:property name="joint_7_axis_xyz" value="0 0 1" />
-    <xacro:property name="joint_7_origin_xyz" value="0 -0.03703 -0.06414" />
-    <xacro:property name="joint_7_origin_rpy" value="${J_PI/3} 0 ${J_PI}" />
-    <xacro:property name="joint_7_lower_limit" value="${-2*J_PI}" />
-    <xacro:property name="joint_7_upper_limit" value="${2*J_PI}" />
-    <xacro:property name="joint_7_velocity_limit" value="${48*J_PI/180}" />
-    <xacro:property name="joint_7_torque_limit" value="20" />
     <xacro:property name="joint_end_effector" value="end_effector_offset" />
     <xacro:property name="joint_end_effector_type" value="fixed" />
@@ -113,5 +102,5 @@
     <xacro:property name="joint_end_effector_origin_xyz" value="0 0 -0.1600" />
     <xacro:property name="joint_end_effector_origin_rpy" value="${J_PI} 0 ${J_PI/2}" />
-    <xacro:macro name="j2n7s300" params="base_parent prefix:=j2n7s300">
+    <xacro:macro name="j2s6s200" params="base_parent prefix:=j2s6s200">
         <xacro:gazebo_config robot_namespace="${prefix}"/>
         <xacro:kinova_armlink link_name="${prefix}_link_base" link_mesh="${link_base_mesh}" mesh_no="${link_base_mesh_no}"/>
@@ -129,9 +118,7 @@
         <xacro:kinova_armlink link_name="${prefix}_link_6" link_mesh="${link_6_mesh}" use_ring_mesh="true" ring_mesh="ring_small" mesh_no="${link_6_mesh_no}"/>
         <xacro:kinova_armjoint joint_name="${prefix}_joint_6" type="${joint_6_type}" parent="${prefix}_link_5" child="${prefix}_link_6" joint_axis_xyz="${joint_6_axis_xyz}" joint_origin_xyz="${joint_6_origin_xyz}" joint_origin_rpy="${joint_6_origin_rpy}" joint_lower_limit="${joint_6_lower_limit}" joint_upper_limit="${joint_6_upper_limit}" joint_velocity_limit="${joint_6_velocity_limit}" joint_torque_limit="${joint_6_torque_limit}"/>
-        <xacro:kinova_armlink link_name="${prefix}_link_7" link_mesh="${link_7_mesh}" use_ring_mesh="true" ring_mesh="ring_small" mesh_no="${link_7_mesh_no}"/>
-        <xacro:kinova_armjoint joint_name="${prefix}_joint_7" type="${joint_7_type}" parent="${prefix}_link_6" child="${prefix}_link_7" joint_axis_xyz="${joint_7_axis_xyz}" joint_origin_xyz="${joint_7_origin_xyz}" joint_origin_rpy="${joint_7_origin_rpy}" joint_lower_limit="${joint_7_lower_limit}" joint_upper_limit="${joint_7_upper_limit}" joint_velocity_limit="${joint_7_velocity_limit}" joint_torque_limit="${joint_7_torque_limit}"/>
         <xacro:kinova_virtual_link link_name="${prefix}_end_effector"/>
-        <xacro:kinova_virtual_joint joint_name="${prefix}_joint_end_effector" type="${joint_end_effector_type}" parent="${prefix}_link_7" child="${prefix}_end_effector" joint_axis_xyz="${joint_end_effector_axis_xyz}" joint_origin_xyz="${joint_end_effector_origin_xyz}" joint_origin_rpy="${joint_end_effector_origin_rpy}" joint_lower_limit="0" joint_upper_limit="0"/>
-        <xacro:kinova_3fingers link_hand="${prefix}_link_7" prefix="${prefix}_"/>
+        <xacro:kinova_virtual_joint joint_name="${prefix}_joint_end_effector" type="${joint_end_effector_type}" parent="${prefix}_link_6" child="${prefix}_end_effector" joint_axis_xyz="${joint_end_effector_axis_xyz}" joint_origin_xyz="${joint_end_effector_origin_xyz}" joint_origin_rpy="${joint_end_effector_origin_rpy}" joint_lower_limit="0" joint_upper_limit="0"/>
+    <xacro:kinova_2fingers link_hand="${prefix}_link_6" prefix="${prefix}_"/>
     </xacro:macro>
 </root>

File: kinova_description/urdf/mico.xacro (robot description, xacro)
@@ -1,4 +1,4 @@
 <?xml version="1.0"?>
-<!-- j2_n7 refers to jaco v2 7DOF non-spherical -->
+<!-- m1_4n refers to mico v1 6DOF non-spherical -->
 <root xmlns:xi="http://www.w3.org/2001/XInclude"
     xmlns:gazebo="http://playerstage.sourceforge.net/gazebo/xmlschema/#gz"
@@ -20,10 +20,7 @@
     <xacro:property name="link_base_mesh" value="base" />
     <xacro:property name="link_1_mesh" value="shoulder" />
-    <xacro:property name="link_2_mesh" value="arm_half_1" />
-    <xacro:property name="link_3_mesh" value="arm_half_2" />
-    <xacro:property name="link_4_mesh" value="forearm" />
-    <xacro:property name="link_5_mesh" value="wrist" />
-    <xacro:property name="link_6_mesh" value="wrist" />
-    <xacro:property name="link_7_mesh" value="hand_3finger" />
+    <xacro:property name="link_2_mesh" value="arm_mico" />
+    <xacro:property name="link_3_mesh" value="forearm_mico" />
+    <xacro:property name="link_4_mesh" value="forearm_mico" />
     <!--Used for conditional arguments for setting inertial parameters
         base 0, shoulder 1, arm 2, forearm 3, wrist 4, arm_mico 5,
@@ -34,10 +31,7 @@
     <xacro:property name="link_base_mesh_no" value="0" />
     <xacro:property name="link_1_mesh_no" value="1" />
-    <xacro:property name="link_2_mesh_no" value="6" />
-    <xacro:property name="link_3_mesh_no" value="7" />
-    <xacro:property name="link_4_mesh_no" value="3" />
-    <xacro:property name="link_5_mesh_no" value="4" />
-    <xacro:property name="link_6_mesh_no" value="4" />
-    <xacro:property name="link_7_mesh_no" value="55" />
+    <xacro:property name="link_2_mesh_no" value="5" />
+    <xacro:property name="link_3_mesh_no" value="10" />
+    <xacro:property name="link_4_mesh_no" value="56" />
     <xacro:property name="joint_base" value="joint_base" />
     <xacro:property name="joint_base_type" value="fixed" />
@@ -58,60 +52,28 @@
     <xacro:property name="joint_2_axis_xyz" value="0 0 1" />
     <xacro:property name="joint_2_origin_xyz" value="0 0.0016 -0.11875" />
-    <xacro:property name="joint_2_origin_rpy" value="-${J_PI/2} 0 ${J_PI}" />
-    <xacro:property name="joint_2_lower_limit" value="${30/180*J_PI}" />
-    <xacro:property name="joint_2_upper_limit" value="${330/180*J_PI}" />
+    <xacro:property name="joint_2_origin_rpy" value="${-J_PI/2} 0 ${J_PI}" />
+    <xacro:property name="joint_2_lower_limit" value="${50/180*J_PI}" />
+    <xacro:property name="joint_2_upper_limit" value="${310/180*J_PI}" />
     <xacro:property name="joint_2_velocity_limit" value="${36*J_PI/180}" />
     <xacro:property name="joint_2_torque_limit" value="80" />
     <xacro:property name="joint_3" value="joint_3" />
-    <xacro:property name="joint_3_type" value="continuous" />
+    <xacro:property name="joint_3_type" value="revolute" />
     <xacro:property name="joint_3_axis_xyz" value="0 0 1" />
-    <xacro:property name="joint_3_origin_xyz" value="0 -0.205 0" />
-    <xacro:property name="joint_3_origin_rpy" value="${J_PI/2} 0 ${J_PI}" />
-    <xacro:property name="joint_3_lower_limit" value="${-5*J_PI/4}" />
-    <xacro:property name="joint_3_upper_limit" value="${1*J_PI/4}" />
+    <xacro:property name="joint_3_origin_xyz" value="0 -0.290 0" />
+    <xacro:property name="joint_3_origin_rpy" value="0 ${J_PI} 0" />
+    <xacro:property name="joint_3_lower_limit" value="${35/180*J_PI}" />
+    <xacro:property name="joint_3_upper_limit" value="${325/180*J_PI}" />
     <xacro:property name="joint_3_velocity_limit" value="${36*J_PI/180}" />
     <xacro:property name="joint_3_torque_limit" value="40" />
     <xacro:property name="joint_4" value="joint_4" />
-    <xacro:property name="joint_4_type" value="revolute" />
+    <xacro:property name="joint_4_type" value="continuous" />
     <xacro:property name="joint_4_axis_xyz" value="0 0 1" />
-    <xacro:property name="joint_4_origin_xyz" value="0 0 -0.205" />
-    <xacro:property name="joint_4_origin_rpy" value="${J_PI/2} 0 ${J_PI}" />
-    <xacro:property name="joint_4_lower_limit" value="${30/180*J_PI}" />
-    <xacro:property name="joint_4_upper_limit" value="${330/180*J_PI}" />
-    <xacro:property name="joint_4_velocity_limit" value="${36*J_PI/180}" />
-    <xacro:property name="joint_4_torque_limit" value="40" />
-    <xacro:property name="joint_5" value="joint_5" />
-    <xacro:property name="joint_5_type" value="continuous" />
-    <xacro:property name="joint_5_axis_xyz" value="0 0 1" />
-    <xacro:property name="joint_5_origin_xyz" value="0 0.2073 -0.0114" />
-    <xacro:property name="joint_5_origin_rpy" value="${-J_PI/2} 0 ${J_PI}" />
-    <xacro:property name="joint_5_lower_limit" value="${-2*J_PI}" />
-    <xacro:property name="joint_5_upper_limit" value="${2*J_PI}" />
-    <xacro:property name="joint_5_velocity_limit" value="${48*J_PI/180}" />
-    <xacro:property name="joint_5_torque_limit" value="20" />
-    <xacro:property name="joint_6" value="joint_6" />
-    <xacro:property name="joint_6_type" value="continuous" />
-    <xacro:property name="joint_6_axis_xyz" value="0 0 1" />
-    <xacro:property name="joint_6_origin_xyz" value="0 -0.03703 -0.06414" />
-    <xacro:property name="joint_6_origin_rpy" value="${J_PI/3} 0 ${J_PI}" />
-    <xacro:property name="joint_6_lower_limit" value="${-2*J_PI}" />
-    <xacro:property name="joint_6_upper_limit" value="${2*J_PI}" />
-    <xacro:property name="joint_6_velocity_limit" value="${48*J_PI/180}" />
-    <xacro:property name="joint_6_torque_limit" value="20" />
-    <xacro:property name="joint_7" value="joint_7" />
-    <xacro:property name="joint_7_type" value="continuous" />
-    <xacro:property name="joint_7_axis_xyz" value="0 0 1" />
-    <xacro:property name="joint_7_origin_xyz" value="0 -0.03703 -0.06414" />
-    <xacro:property name="joint_7_origin_rpy" value="${J_PI/3} 0 ${J_PI}" />
-    <xacro:property name="joint_7_lower_limit" value="${-2*J_PI}" />
-    <xacro:property name="joint_7_upper_limit" value="${2*J_PI}" />
-    <xacro:property name="joint_7_velocity_limit" value="${48*J_PI/180}" />
-    <xacro:property name="joint_7_torque_limit" value="20" />
-    <xacro:property name="joint_end_effector" value="end_effector_offset" />
-    <xacro:property name="joint_end_effector_type" value="fixed" />
-    <xacro:property name="joint_end_effector_axis_xyz" value="0 0 0" />
-    <xacro:property name="joint_end_effector_origin_xyz" value="0 0 -0.1600" />
-    <xacro:property name="joint_end_effector_origin_rpy" value="${J_PI} 0 ${J_PI/2}" />
-    <xacro:macro name="j2n7s300" params="base_parent prefix:=j2n7s300">
+    <xacro:property name="joint_4_origin_xyz" value="0 0.1231 -0.0086" />
+    <xacro:property name="joint_4_origin_rpy" value="${-J_PI/2} 0 ${J_PI}" />
+    <xacro:property name="joint_4_lower_limit" value="${-2*J_PI}" />
+    <xacro:property name="joint_4_upper_limit" value="${2*J_PI}" />
+    <xacro:property name="joint_4_velocity_limit" value="${48*J_PI/180}" />
+    <xacro:property name="joint_4_torque_limit" value="20" />
+    <xacro:macro name="mico" params="base_parent prefix:=mico">
         <xacro:gazebo_config robot_namespace="${prefix}"/>
         <xacro:kinova_armlink link_name="${prefix}_link_base" link_mesh="${link_base_mesh}" mesh_no="${link_base_mesh_no}"/>
@@ -125,13 +87,4 @@
         <xacro:kinova_armlink link_name="${prefix}_link_4" link_mesh="${link_4_mesh}" use_ring_mesh="true" ring_mesh="ring_small" mesh_no="${link_4_mesh_no}"/>
         <xacro:kinova_armjoint joint_name="${prefix}_joint_4" type="${joint_4_type}" parent="${prefix}_link_3" child="${prefix}_link_4" joint_axis_xyz="${joint_4_axis_xyz}" joint_origin_xyz="${joint_4_origin_xyz}" joint_origin_rpy="${joint_4_origin_rpy}" joint_lower_limit="${joint_4_lower_limit}" joint_upper_limit="${joint_4_upper_limit}" joint_velocity_limit="${joint_4_velocity_limit}" joint_torque_limit="${joint_4_torque_limit}"/>
-        <xacro:kinova_armlink link_name="${prefix}_link_5" link_mesh="${link_5_mesh}" use_ring_mesh="true" ring_mesh="ring_small" mesh_no="${link_5_mesh_no}"/>
-        <xacro:kinova_armjoint joint_name="${prefix}_joint_5" type="${joint_5_type}" parent="${prefix}_link_4" child="${prefix}_link_5" joint_axis_xyz="${joint_5_axis_xyz}" joint_origin_xyz="${joint_5_origin_xyz}" joint_origin_rpy="${joint_5_origin_rpy}" joint_lower_limit="${joint_5_lower_limit}" joint_upper_limit="${joint_5_upper_limit}" joint_velocity_limit="${joint_5_velocity_limit}" joint_torque_limit="${joint_5_torque_limit}"/>
-        <xacro:kinova_armlink link_name="${prefix}_link_6" link_mesh="${link_6_mesh}" use_ring_mesh="true" ring_mesh="ring_small" mesh_no="${link_6_mesh_no}"/>
-        <xacro:kinova_armjoint joint_name="${prefix}_joint_6" type="${joint_6_type}" parent="${prefix}_link_5" child="${prefix}_link_6" joint_axis_xyz="${joint_6_axis_xyz}" joint_origin_xyz="${joint_6_origin_xyz}" joint_origin_rpy="${joint_6_origin_rpy}" joint_lower_limit="${joint_6_lower_limit}" joint_upper_limit="${joint_6_upper_limit}" joint_velocity_limit="${joint_6_velocity_limit}" joint_torque_limit="${joint_6_torque_limit}"/>
-        <xacro:kinova_armlink link_name="${prefix}_link_7" link_mesh="${link_7_mesh}" use_ring_mesh="true" ring_mesh="ring_small" mesh_no="${link_7_mesh_no}"/>
-        <xacro:kinova_armjoint joint_name="${prefix}_joint_7" type="${joint_7_type}" parent="${prefix}_link_6" child="${prefix}_link_7" joint_axis_xyz="${joint_7_axis_xyz}" joint_origin_xyz="${joint_7_origin_xyz}" joint_origin_rpy="${joint_7_origin_rpy}" joint_lower_limit="${joint_7_lower_limit}" joint_upper_limit="${joint_7_upper_limit}" joint_velocity_limit="${joint_7_velocity_limit}" joint_torque_limit="${joint_7_torque_limit}"/>
-        <xacro:kinova_virtual_link link_name="${prefix}_end_effector"/>
-        <xacro:kinova_virtual_joint joint_name="${prefix}_joint_end_effector" type="${joint_end_effector_type}" parent="${prefix}_link_7" child="${prefix}_end_effector" joint_axis_xyz="${joint_end_effector_axis_xyz}" joint_origin_xyz="${joint_end_effector_origin_xyz}" joint_origin_rpy="${joint_end_effector_origin_rpy}" joint_lower_limit="0" joint_upper_limit="0"/>
-        <xacro:kinova_3fingers link_hand="${prefix}_link_7" prefix="${prefix}_"/>
     </xacro:macro>
 </root>
